Commit message: added forward looking sonar

File: robots/rexrov2_iiwa14_merged.xacro (robot description, xacro)
@@ -22,4 +22,21 @@
   <xacro:include filename="$(find rexrov2_description)/urdf/rexrov2.gazebo.xacro"/>
   <xacro:include filename="$(find rexrov2_iiwa14)/urdf/iiwa14_uuv_merged.xacro" />
+  <xacro:forward_looking_sonar
+      namespace="$(arg namespace)"
+      suffix="down"
+      parent_link="$(arg namespace)/base_link"
+      topic="forward_sonar"
+      mass="0.015"
+      update_rate="40"
+      samples="100"
+        fov="1.54719755"
+        width="768"
+        height="492">
+      <inertia ixx="0.00001" ixy="0.0" ixz="0.0" iyy="0.00001" iyz="0.0" izz="0.00001" />
+      <!--origin xyz="0.83 0 -0.22" rpy="0 ${0.2*pi} 0" /-->
+      <origin xyz="1.15 0 0.4" rpy="0 0.3 0"/>
+      <visual>
+      </visual>
+  </xacro:forward_looking_sonar>
   <!-- Create the ROV -->
   <xacro:rexrov2_base

Commit message: changes to FLS position and added multibeam sonar

File: robots/rexrov2_iiwa14_merged.xacro (robot description, xacro)
@@ -35,8 +35,11 @@
       <inertia ixx="0.00001" ixy="0.0" ixz="0.0" iyy="0.00001" iyz="0.0" izz="0.00001" />
       <!--origin xyz="0.83 0 -0.22" rpy="0 ${0.2*pi} 0" /-->
-      <origin xyz="1.15 0 0.4" rpy="0 0.3 0"/>
+      <origin xyz="1.15 0 -0.6" rpy="0 0.3 0"/>
       <visual>
       </visual>
   </xacro:forward_looking_sonar>
+  <xacro:forward_multibeam_sonar_m450_130 namespace="$(arg namespace)" parent_link="$(arg namespace)/base_link">
+    <origin xyz="1.35 0 0.9" rpy="0 0 0"/>
+  </xacro:forward_multibeam_sonar_m450_130>
   <!-- Create the ROV -->
   <xacro:rexrov2_base

Commit message: changed position of FLS and Forward multibeam

File: robots/rexrov2_iiwa14_merged.xacro (robot description, xacro)
@@ -35,10 +35,10 @@
       <inertia ixx="0.00001" ixy="0.0" ixz="0.0" iyy="0.00001" iyz="0.0" izz="0.00001" />
       <!--origin xyz="0.83 0 -0.22" rpy="0 ${0.2*pi} 0" /-->
-      <origin xyz="1.15 0 -0.6" rpy="0 0.3 0"/>
+      <origin xyz="1.15 0 0.4" rpy="0 0.3 0"/>
       <visual>
       </visual>
   </xacro:forward_looking_sonar>
   <xacro:forward_multibeam_sonar_m450_130 namespace="$(arg namespace)" parent_link="$(arg namespace)/base_link">
-    <origin xyz="1.35 0 0.9" rpy="0 0 0"/>
+    <origin xyz="1.35 0 0.6" rpy="0 0 0"/>
   </xacro:forward_multibeam_sonar_m450_130>
   <!-- Create the ROV -->
@@ -71,4 +71,6 @@
         <robotNamespace>/$(arg namespace)</robotNamespace>
         <robotParam>/$(arg namespace)/robot_description</robotParam>
+        <robotSimType>gazebo_ros_control/DefaultRobotHWSim</robotSimType>
+        <legacyModeNS>true</legacyModeNS>
       </plugin>
    </gazebo>

Commit message: iiwa initial position 000000

File: robots/rexrov2_iiwa14_merged.xacro (robot description, xacro)
@@ -62,4 +62,5 @@
 <!--  </xacro:iiwa14>-->
 <xacro:iiwa14   parent="$(arg namespace)/base_link" hardware_interface="PositionJointInterface" robot_name="iiwa" tool_l="$(arg tool_l)">
+    <!-- <origin xyz="1.22 0 -0.75" rpy="0 0 3.1416"/> -->
     <origin xyz="1.22 0 -0.75" rpy="0 0 3.1416"/>
   </xacro:iiwa14>

File: urdf/iiwa14_uuv_merged.xacro (robot description, xacro)
@@ -158,5 +158,5 @@
       <parent link="${robot_name}_link_3"/>
       <child link="${robot_name}_link_4"/>
-      <origin xyz="0 0 0.2155" rpy="${PI / 2} ${-PI / 2} 0"/> <!--${PI / 2} 0 0 -->
+      <origin xyz="0 0 0.2155" rpy="${PI / 2} 0 0"/> <!--original:"${PI / 2} 0 0", rotated:"${PI / 2} ${-PI / 2} 0"-->
       <axis xyz="0 0 1"/>
       <limit lower="${-120 * PI / 180}" upper="${120 * PI / 180}"
